File: _autosave-bakeneko60tho.kicad_pcb (KiCad board)
At the start: 2 copper layers, 285.8 x 95.2 mm, 160 parts, among them J1 Conn_01x04_Male, SW1 SW_Push, U1 ATmega32U4-AU, Y1 16MHz

Commit message: complete routing
finishing the routing
Parts:
- moved D41 10.3 mm to (204.0, 60.3), turned to 90 degrees
Connections:
- U1 pad 10: Net-(U1-Pad10) -> COL8
- U1 pad 11: Net-(U1-Pad11) -> COL9
- U1 pad 12: Net-(U1-Pad12) -> COL10
- U1 pad 18: Net-(U1-Pad18) -> COL14
- U1 pad 19: Net-(U1-Pad19) -> COL13
- U1 pad 20: Net-(U1-Pad20) -> COL12
- U1 pad 21: Net-(U1-Pad21) -> COL11
- U1 pad 26: Net-(U1-Pad26) -> ROW1
- U1 pad 27: Net-(U1-Pad27) -> ROW0
- U1 pad 28: Net-(U1-Pad28) -> ROW4
- U1 pad 29: Net-(U1-Pad29) -> ROW3
- U1 pad 30: Net-(U1-Pad30) -> ROW2
- U1 pad 8: Net-(U1-Pad8) -> COL6
- U1 pad 9: Net-(U1-Pad9) -> COL7
Routing:
- net ROW4: track 274.0 -> 374.4 mm, vias 0 -> 2
- net COL6: track 66.1 -> 153.7 mm, vias 0 -> 1
- net COL14: track 88.1 -> 158.4 mm
- net COL7: track 88.1 -> 156.6 mm, vias 0 -> 1
- net COL13: track 83.1 -> 133.3 mm
- net COL8: track 88.1 -> 137.5 mm, vias 0 -> 1
- net ROW1: track 237.8 -> 286.0 mm, vias 0 -> 2
- net ROW3: track 274.1 -> 322.0 mm, vias 0 -> 2
- net ROW0: track 275.0 -> 311.6 mm, vias 0 -> 2
- net COL9: track 88.1 -> 118.4 mm, vias 0 -> 1
- net COL12: track 87.1 -> 117.1 mm
- net ROW2: track 277.0 -> 295.0 mm, vias 0 -> 2
- net COL10: track 88.1 -> 102.5 mm
- net Net-(U1-Pad30): track 7.48 -> 0.00 mm
- net Net-(U1-Pad29): track 7.34 -> 0.00 mm
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