File: bakeneko60tho.kicad_pcb (KiCad board)
At the start: 2 copper layers, 160 parts, among them J1 Conn_01x04_Male, SW1 SW_Push, U1 ATmega32U4-AU, Y1 16MHz

Commit message: complete routing
finishing the routing
Parts:
- C1, C2, C3, C4, C5, C6, C7, D1, D10, D11, D12, D13, D14, D15, D16, D17, D18, D19, D2, D20, D21, D22, D23, D24, D25, D26, D27, D28, D29, D3, D30, D31, D32, D33, D34, D35, D36, D37, D38, D39, D4, D40, D41, D42, D43, D44, D45, D46, D47, D48, D49, D5, D50, D51, D52, D53, D54, D55, D56, D57, D58, D59, D6, D60, D61, D62, D63, D64, D65, D66, D67, D68, D69, D7, D70, D71, D72, D8, D9, F1, J1, R1, R2, R3, R4, SW1, U1, Y1: moved to B.Cu
- moved C3 332.8 mm to (217.5, 27.0), turned to 270 degrees
- moved C5 331.2 mm to (232.3, 46.1), turned to 90 degrees
- moved D72 328.2 mm to (296.9, 98.4)
- moved C6 319.5 mm to (212.7, 49.2), turned to 180 degrees
- moved C7 316.9 mm to (211.3, 54.8), turned to 270 degrees
- moved C4 310.6 mm to (223.8, 62.2), turned to 180 degrees
- moved C2 285.9 mm to (227.0, 27.0), turned to 90 degrees
- moved F1 260.9 mm to (77.7, 52.8)
- moved C1 252.0 mm to (217.5, 31.8), turned to 90 degrees
- moved R2 242.0 mm to (75.7, 30.1), turned to 180 degrees
- moved Y1 233.3 mm to (222.1, 27.0), turned to 180 degrees
- moved R1 227.2 mm to (75.7, 33.4), turned to 180 degrees
- moved R3 195.3 mm to (214.0, 31.8), turned to 90 degrees
- moved U1 192.4 mm to (223.1, 49.8), turned to 0 degrees
- moved R4 183.8 mm to (231.8, 55.6), turned to 90 degrees
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Connections:
- F1 pad 1: +5V -> VCC
- F1 pad 2: VCC -> +5V
- J1 pad 1: VCC -> GND
- J1 pad 2: D- -> D+
- J1 pad 3: D+ -> D-
- J1 pad 4: GND -> VCC
- U1 pad 10: COL12 -> COL8
- U1 pad 11: COL11 -> COL9
- U1 pad 12: COL7 -> COL10
- U1 pad 18: COL6 -> COL14
- U1 pad 19: COL5 -> COL13
- U1 pad 20: COL4 -> COL12
- U1 pad 21: COL3 -> COL11
- U1 pad 26: COL2 -> Net-(U1-Pad26)
- U1 pad 27: COL1 -> Net-(U1-Pad27)
- U1 pad 28: COL10 -> Net-(U1-Pad28)
- U1 pad 29: COL9 -> Net-(U1-Pad29)
- U1 pad 30: COL8 -> Net-(U1-Pad30)
- U1 pad 36: ROW4 -> Net-(U1-Pad36)
- U1 pad 37: ROW3 -> Net-(U1-Pad37)
- U1 pad 38: ROW2 -> Net-(U1-Pad38)
- U1 pad 39: ROW1 -> Net-(U1-Pad39)
- U1 pad 40: ROW0 -> Net-(U1-Pad40)
- U1 pad 41: COL0 -> Net-(U1-Pad41)
- U1 pad 8: COL14 -> COL6
- U1 pad 9: COL13 -> COL7
Routing:
- net ROW0: track 0.00 -> 275.0 mm
- net ROW1: track 0.00 -> 274.6 mm, vias 0 -> 2
- net ROW3: track 0.00 -> 274.1 mm
- net ROW4: track 0.00 -> 274.0 mm
- net ROW2: track 0.00 -> 271.8 mm
- net GND: track 0.00 -> 256.2 mm
- net +5V: track 0.00 -> 244.2 mm, vias 0 -> 6
- net Net-(R2-Pad1): track 0.00 -> 160.3 mm, vias 0 -> 2
- net Net-(R1-Pad1): track 0.00 -> 160.2 mm, vias 0 -> 2
- net COL14: track 0.00 -> 158.4 mm
- net COL7: track 0.00 -> 156.6 mm, vias 0 -> 1
- net COL6: track 0.00 -> 153.7 mm, vias 0 -> 1
- net COL8: track 0.00 -> 137.5 mm, vias 0 -> 1
- net COL13: track 0.00 -> 133.3 mm
- net COL9: track 0.00 -> 118.4 mm, vias 0 -> 1
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Other:
- board outline added: 285.8 x 95.2 mm
- net class Power added: clearance 0.2, trace_width 0.381, via_dia 0.8, via_drill 0.4

Commit message: fix routing
fix routing bugs
Parts:
- added J2: D+, Connector_PinHeader_1.00mm:PinHeader_1x01_P1.00mm_Vertical, B.Cu at (69.8, 30.5)
- added J3: D-, Connector_PinHeader_1.00mm:PinHeader_1x01_P1.00mm_Vertical, B.Cu at (69.8, 33.0)
- added J4: vcc, Connector_PinHeader_1.00mm:PinHeader_1x01_P1.00mm_Vertical, B.Cu at (69.8, 35.4)
- J1: value Conn_01x04_Male -> GND; footprint Connector_PinHeader_1.00mm:PinHeader_1x04_P1.00mm_Horizontal -> Connector_PinHeader_1.00mm:PinHeader_1x01_P1.00mm_Vertical
- moved J1 2.16 mm to (69.8, 28.1), turned to 90 degrees
Connections:
- U1 pad 26: Net-(U1-Pad26) -> ROW1
- U1 pad 27: Net-(U1-Pad27) -> ROW0
- U1 pad 28: Net-(U1-Pad28) -> ROW4
- U1 pad 29: Net-(U1-Pad29) -> ROW3
- U1 pad 30: Net-(U1-Pad30) -> ROW2
- U1 pad 36: Net-(U1-Pad36) -> COL0
- U1 pad 37: Net-(U1-Pad37) -> COL1
- U1 pad 38: Net-(U1-Pad38) -> COL2
- U1 pad 39: Net-(U1-Pad39) -> COL3
- U1 pad 40: Net-(U1-Pad40) -> COL4
- U1 pad 41: Net-(U1-Pad41) -> COL5
Routing:
- net COL0: track 88.1 -> 305.8 mm, vias 0 -> 3
- net COL1: track 88.1 -> 285.6 mm, vias 0 -> 3
- net COL2: track 87.5 -> 264.7 mm, vias 0 -> 3
- net COL3: track 88.1 -> 244.7 mm, vias 0 -> 3
- net COL4: track 88.1 -> 225.8 mm, vias 0 -> 3
- net COL5: track 89.1 -> 206.0 mm, vias 0 -> 3
- net ROW4: track 274.0 -> 374.4 mm, vias 0 -> 2
- net ROW3: track 274.1 -> 322.0 mm, vias 0 -> 2
- net ROW2: track 271.8 -> 295.0 mm, vias 0 -> 2
- net ROW1: track 274.6 -> 286.0 mm
- net Net-(U1-Pad30): track 7.48 -> 0.00 mm
- net Net-(U1-Pad29): track 7.34 -> 0.00 mm
- net Net-(U1-Pad28): track 7.19 -> 0.00 mm
- net Net-(U1-Pad27): track 7.05 -> 0.00 mm
- net Net-(U1-Pad26): track 6.89 -> 0.00 mm
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- added copper zone on B.Cu, net GND
