File: bakeneko60tho.kicad_pcb (KiCad board)
At the start: 2 copper layers, 285.8 x 95.2 mm, 160 parts, among them J1 Conn_01x04, SW1 SW_Push, U1 ATmega32U4-AU, Y1 16MHz

Commit message: clean up routing
Parts:
- moved R1 32.3 mm to (108.0, 32.8)
- moved R2 32.3 mm to (108.0, 30.7)
- moved F1 26.0 mm to (95.1, 33.5)
- moved R4 2.23 mm to (231.9, 53.3), turned to 270 degrees
- moved J1 1.77 mm to (66.7, 31.8)
- moved C7 1.43 mm to (212.6, 54.1)
- moved C6 0.88 mm to (213.5, 49.7), turned to 270 degrees
- moved C5 0.72 mm to (231.8, 45.6)
- moved C4 0.32 mm to (223.8, 61.9)
- turned SW1 to 180 degrees
Connections:
- U1 pad 10: COL8 -> COL7
- U1 pad 11: COL9 -> COL6
- U1 pad 36: COL0 -> COL5
- U1 pad 37: COL1 -> COL4
- U1 pad 38: COL2 -> COL3
- U1 pad 39: COL3 -> COL2
- U1 pad 40: COL4 -> COL1
- U1 pad 41: COL5 -> COL0
- U1 pad 8: COL6 -> COL9
- U1 pad 9: COL7 -> COL8
Routing:
- net ROW2: track 295.0 -> 341.4 mm, vias 2 -> 4
- net ROW0: track 316.2 -> 356.8 mm
- net D-: track 3.92 -> 42.6 mm
- net D+: track 3.95 -> 42.6 mm
- net ROW3: track 322.0 -> 356.1 mm
- net Net-(R1-Pad1): track 160.2 -> 127.9 mm
- net Net-(R2-Pad1): track 160.3 -> 128.2 mm
- net COL11: track 94.7 -> 111.1 mm
- net GND: track 254.7 -> 269.1 mm, vias 0 -> 2
- net Net-(R3-Pad1): track 32.4 -> 25.5 mm
- net VCC: track 23.3 -> 30.0 mm, vias 1 -> 0
- net COL0: track 305.8 -> 299.7 mm, vias 3 -> 1
- net COL1: track 285.6 -> 281.6 mm, vias 3 -> 1
- net COL5: track 206.0 -> 209.9 mm, vias 3 -> 1
- net ROW1: track 286.0 -> 288.4 mm
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